Commit message: improved path planning parameters and updated urdf

File: src/rosie_description/urdf/macros.xacro (robot description, xacro)
@@ -49,7 +49,7 @@
     </gazebo>
     <joint name="${lr}_wheel_hinge" type="continuous">
-      <parent link="chassis"/>
+      <parent link="base_link"/>
       <child link="${lr}_wheel"/>
-    <origin xyz="${-wheelPos+chassisLength/2} ${tY*wheelWidth/2+tY*chassisWidth/2} ${wheelRadius}" rpy="0 0 0" />
+    <origin xyz="${-wheelPos+base_linkLength/2} ${tY*wheelWidth/2+tY*base_linkWidth/2} ${wheelRadius}" rpy="0 0 0" />
       <axis xyz="0 1 0" rpy="0 0 0" />
       <limit effort="10000" velocity="10000"/>

File: src/rosie_description/urdf/rosie.xacro (robot description, xacro)
@@ -1,4 +1,4 @@
 <?xml version='1.0'?>
-<robot name="myrobot" xmlns:xacro="http://www.ros.org/wiki/xacro">
+<robot name="rosie" xmlns:xacro="http://www.ros.org/wiki/xacro">
   <xacro:property name="cameraSize" value="0.05"/>
   <xacro:property name="cameraMass" value="0.1"/>
@@ -6,32 +6,44 @@
   <xacro:include filename="$(find rosie_description)/urdf/materials.xacro" />
   <xacro:include filename="$(find rosie_description)/urdf/macros.xacro" />
-  <link name='chassis'>
-    <pose>0 0 0.1 0 0 0</pose>
+  <link name='base_link'>
     <inertial>
-      <mass value="15.0"/>
-      <origin xyz="0.0 0 0.1" rpy=" 0 0 0"/>
-      <inertia
-          ixx="0.1" ixy="0" ixz="0"
-          iyy="0.1" iyz="0"
-          izz="0.1"
+      <mass value="2.0"/>
+      <!-- Assume Moment of inertia is from a solid cylinder for now -->
+	  <inertia
+          ixx="0.0209" ixy="0" ixz="0"
+          iyy="0.0209" iyz="0"
+          izz="0.04"
       />
     </inertial>
     <collision name='collision'>
       <geometry>
-        <box size=".4 .2 .1"/>
+        <cylinder radius="0.2" length="0.075"/>
       </geometry>
     </collision>
-    <visual name='chassis_visual'>
-      <origin xyz="0 0 0" rpy=" 0 0 0"/>
+    <visual name='base_link_visual'>
       <geometry>
-        <box size=".4 .2 .1"/>
+        <cylinder radius="0.2" length="0.075"/>
       </geometry>
     </visual>
-    <collision name='caster_collision'>
-      <origin xyz="-0.15 0 -0.05" rpy=" 0 0 0"/>
+  </link>
+  <link name='caster'>
+    <inertial>
+      <mass value="0.010"/>
+	  <inertia
+          ixx="0.0" ixy="0" ixz="0"
+          iyy="0.0" iyz="0"
+          izz="0.0"
+      />
+    </inertial>
+    <visual name='caster_visual'>
       <geometry>
-        <sphere radius="0.05"/>
+        <sphere radius="0.01"/>
       </geometry>
-      <surface>
+    </visual>
+    <collision name='collision'>
+      <geometry>
+        <sphere radius="0.01"/>
+      </geometry>
+      <!--surface>
         <friction>
           <ode>
@@ -42,41 +54,17 @@
           </ode>
         </friction>
-      </surface>
+      </surface-->
     </collision>
-    <visual name='caster_visual'>
-      <origin xyz="-0.15 0 -0.05" rpy=" 0 0 0"/>
-      <geometry>
-        <sphere radius="0.05"/>
-      </geometry>
-    </visual>
-    <collision name='caster_front_collision'>
-      <origin xyz="0.15 0 -0.05" rpy=" 0 0 0"/>
-      <geometry>
-        <sphere radius="0.05"/>
-      </geometry>
-      <surface>
-        <friction>
-          <ode>
-            <mu>0</mu>
-            <mu2>0</mu2>
-            <slip1>1.0</slip1>
-            <slip2>1.0</slip2>
-          </ode>
-        </friction>
-      </surface>
-    </collision>
-    <visual name='caster_front_visual'>
-      <origin xyz="0.15 0 -0.05" rpy=" 0 0 0"/>
-      <geometry>
-        <sphere radius="0.05"/>
-      </geometry>
-    </visual>
   </link>
+  <joint type="fixed" name="caster_joint">
+    <origin xyz="-0.15 0 -0.0375" rpy="0 0 0"/>
+    <child link="caster"/>
+    <parent link="base_link"/>
+  </joint>
   <link name="left_wheel">
-    <!--origin xyz="0.1 0.13 0.1" rpy="0 1.5707 1.5707"/-->
     <collision name="collision">
       <origin xyz="0 0 0" rpy="0 1.5707 1.5707"/>
       <geometry>
-        <cylinder radius="0.1" length="0.05"/>
+        <cylinder radius="0.032" length="0.02"/>
       </geometry>
     </collision>
@@ -84,5 +72,5 @@
       <origin xyz="0 0 0" rpy="0 1.5707 1.5707"/>
       <geometry>
-        <cylinder radius="0.1" length="0.05"/>
+        <cylinder radius="0.032" length="0.02"/>
       </geometry>
     </visual>
@@ -91,15 +79,22 @@
       <mass value="5"/>
       <inertia
-        ixx=".1" ixy="0.0" ixz="0.0"
-        iyy=".1" iyz="0.0"
-        izz=".1"/>
+        ixx=".01167" ixy="0.0" ixz="0.0"
+        iyy=".01167" iyz="0.0"
+        izz=".01885"/>
     </inertial>
   </link>
+  <joint type="continuous" name="left_wheel_hinge">
+    <origin xyz="0.05 0.15 -0.0145" rpy="0 0 0"/>
+    <child link="left_wheel"/>
+    <parent link="base_link"/>
+    <axis xyz="0 1 0" rpy="0 0 0"/>
+    <limit effort="10000" velocity="1000"/>
+    <joint_properties damping="1.0" friction="1.0"/>
+  </joint>
   <link name="right_wheel">
-    <!--origin xyz="0.1 -0.13 0.1" rpy="0 1.5707 1.5707"/-->
     <collision name="collision">
       <origin xyz="0 0 0" rpy="0 1.5707 1.5707"/>
       <geometry>
-        <cylinder radius="0.1" length="0.05"/>
+        <cylinder radius="0.032" length="0.02"/>
       </geometry>
     </collision>
@@ -107,5 +102,5 @@
       <origin xyz="0 0 0" rpy="0 1.5707 1.5707"/>
       <geometry>
-        <cylinder radius="0.1" length="0.05"/>
+        <cylinder radius="0.032" length="0.02"/>
       </geometry>
     </visual>
@@ -114,28 +109,18 @@
       <mass value="5"/>
       <inertia
-        ixx=".1" ixy="0.0" ixz="0.0"
-        iyy=".1" iyz="0.0"
-        izz=".1"/>
+        ixx=".01167" ixy="0.0" ixz="0.0"
+        iyy=".01167" iyz="0.0"
+        izz=".01885"/>
     </inertial>
   </link>
-  <joint type="continuous" name="left_wheel_hinge">
-    <origin xyz="0 0.15 0" rpy="0 0 0"/>
-    <!--origin xyz="0.1 0.13 0" rpy="0 1.5707 1.5707"/-->
-    <child link="left_wheel"/>
-    <parent link="chassis"/>
+  <joint type="continuous" name="right_wheel_hinge">
+    <origin xyz="0.05 -0.15 -0.0145" rpy="0 0 0"/>
+    <child link="right_wheel"/>
+    <parent link="base_link"/>
     <axis xyz="0 1 0" rpy="0 0 0"/>
     <limit effort="10000" velocity="1000"/>
     <joint_properties damping="1.0" friction="1.0"/>
   </joint>
-  <joint type="continuous" name="right_wheel_hinge">
-    <origin xyz="0 -0.15 0" rpy="0 0 0"/>
-    <!--origin xyz="0.1 -0.13 0" rpy="0 1.5707 1.5707"/-->
-    <child link="right_wheel"/>
-    <parent link="chassis"/>
-    <axis xyz="0 1 0" rpy="0 0 0"/>
-    <limit effort="10000" velocity="1000"/>
-    <joint_properties damping="1.0" friction="1.0"/>
-  </joint>
-  <link name="camera">
+  <!--link name="camera">
     <collision>
       <origin xyz="0 0 0" rpy="0 0 0"/>
@@ -161,11 +146,11 @@
     <axis xyz="0 1 0" />
     <origin xyz=".2 0 0" rpy="0 0 0"/>
-    <parent link="chassis"/>
+    <parent link="base_link"/>
     <child link="camera"/>
-  </joint>
+  </joint-->
   <joint name="hokuyo_joint" type="fixed">
     <axis xyz="0 1 0" />
-    <origin xyz=".15 0 .1" rpy="0 0 0"/>
-    <parent link="chassis"/>
+    <origin xyz="0 0 .075" rpy="0 0 0"/>
+    <parent link="base_link"/>
     <child link="hokuyo"/>
   </joint>

Commit message: fixed friction issues with URDF model and improved pathing params

File: src/rosie_description/urdf/macros.xacro (robot description, xacro)
@@ -1,69 +1,64 @@
 <?xml version="1.0"?>
 <robot>
-  <!--macro name="cylinder_inertia" params="m r h">
-    <inertia  ixx="${m*(3*r*r+h*h)/12}" ixy = "0" ixz = "0"
-      iyy="${m*(3*r*r+h*h)/12}" iyz = "0"
-      izz="${m*r*r/2}"
-    />
-  </macro>
-  <macro name="box_inertia" params="m x y z">
-    <inertia  ixx="${m*(y*y+z*z)/12}" ixy = "0" ixz = "0"
-      iyy="${m*(x*x+z*z)/12}" iyz = "0"
-      izz="${m*(x*x+z*z)/12}"
-    />
-  </macro>
-  <macro name="sphere_inertia" params="m r">
-    <inertia  ixx="${2*m*r*r/5}" ixy = "0" ixz = "0"
-      iyy="${2*m*r*r/5}" iyz = "0"
-      izz="${2*m*r*r/5}"
-    />
-  </macro>
-  <macro name="wheel" params="lr tY">
-    <link name="${lr}_wheel">
-      <collision>
-        <origin xyz="0 0 0" rpy="0 ${PI/2} ${PI/2}" />
-        <geometry>
-          <cylinder length="${wheelWidth}" radius="${wheelRadius}"/>
-        </geometry>
-      </collision>
-      <visual>
-        <origin xyz="0 0 0" rpy="0 ${PI/2} ${PI/2}" />
-        <geometry>
-          <cylinder length="${wheelWidth}" radius="${wheelRadius}"/>
-        </geometry>
-        <material name="black"/>
-      </visual>
-      <inertial>
-        <origin xyz="0 0 0" rpy="0 ${PI/2} ${PI/2}" />
-        <mass value="${wheelMass}"/>
-        <cylinder_inertia m="${wheelMass}" r="${wheelRadius}" h="${wheelWidth}"/>
-      </inertial>
-    </link>
-    <gazebo reference="${lr}_wheel">
-      <mu1 value="1.0"/>
-      <mu2 value="1.0"/>
-      <kp  value="10000000.0" />
-      <kd  value="1.0" />
-      <fdir1 value="1 0 0"/>
-      <material>Gazebo/Black</material>
-    </gazebo>
-    <joint name="${lr}_wheel_hinge" type="continuous">
-      <parent link="base_link"/>
-      <child link="${lr}_wheel"/>
-    <origin xyz="${-wheelPos+base_linkLength/2} ${tY*wheelWidth/2+tY*base_linkWidth/2} ${wheelRadius}" rpy="0 0 0" />
-      <axis xyz="0 1 0" rpy="0 0 0" />
-      <limit effort="10000" velocity="10000"/>
-      <joint_properties damping="0.0" friction="0.0"/>
-    </joint>
-    <transmission name="${lr}_trans">
-      <type>transmission_interface/SimpleTransmission</type>
-      <joint name="${lr}_wheel_hinge">
-        <hardwareInterface>EffortJointInterface</hardwareInterface>
-      </joint>
-      <actuator name="${lr}Motor">
-        <hardwareInterface>EffortJointInterface</hardwareInterface>
-        <mechanicalReduction>10</mechanicalReduction>
-      </actuator>
-    </transmission>
-  </macro-->
+     <macro name="cylinder_inertia" params="m r h">
+        <inertia  ixx="${m*(3*r*r+h*h)/12}" ixy = "0" ixz = "0"
+                  iyy="${m*(3*r*r+h*h)/12}" iyz = "0"
+                  izz="${m*r*r/2}" />
+      </macro>
+      <macro name="box_inertia" params="m x y z">
+        <inertia  ixx="${m*(y*y+z*z)/12}" ixy = "0" ixz = "0"
+                  iyy="${m*(x*x+z*z)/12}" iyz = "0"
+                  izz="${m*(x*x+z*z)/12}" />
+      </macro>
+      <macro name="sphere_inertia" params="m r">
+        <inertia  ixx="${2*m*r*r/5}" ixy = "0" ixz = "0"
+                  iyy="${2*m*r*r/5}" iyz = "0"
+                  izz="${2*m*r*r/5}" />
+      </macro>
+     <macro name="wheel" params="lr tY">
+       <link name="${lr}_wheel">
+        <collision>
+          <origin xyz="0 0 0" rpy="0 ${PI/2} ${PI/2}" />
+          <geometry>
+           <cylinder length="${wheelWidth}" radius="${wheelRadius}"/>
+          </geometry>
+        </collision>
+        <visual>
+          <origin xyz="0 0 0" rpy="0 ${PI/2} ${PI/2}" />
+          <geometry>
+           <cylinder length="${wheelWidth}" radius="${wheelRadius}"/>
+          </geometry>
+          <material name="black"/>
+        </visual>
+        <inertial>
+          <origin xyz="0 0 0" rpy="0 ${PI/2} ${PI/2}" />
+          <mass value="${wheelMass}"/>
+          <cylinder_inertia m="${wheelMass}" r="${wheelRadius}" h="${wheelWidth}"/>
+        </inertial>
+       </link>
+        <!--gazebo reference="${lr}_wheel">
+          <mu1 value="1.0"/>
+          <mu2 value="1.0"/>
+          <kp  value="10000000.0" />
+          <kd  value="1.0" />
+          <fdir1 value="1 0 0"/>
+          <material>Gazebo/Black</material>
+        </gazebo-->
+       <joint name="${lr}_wheel_hinge" type="continuous">
+          <parent link="base_link"/>
+          <child link="${lr}_wheel"/>
+          <origin xyz="${+wheelBase/2-chassisRadius/2} ${tY*wheelBase/2} ${wheelRadius-(chassisHeight/2+groundClearance)}" rpy="0 0 0" />
+          <axis xyz="0 1 0" rpy="0 0 0" />
+          <limit effort="100" velocity="100"/>
+          <joint_properties damping="0.0" friction="0.0"/>
+        </joint>
+      <!--transmission name="${lr}_trans">
+        <type>transmission_interface/SimpleTransmission</type>
+        <joint name="${lr}_wheel_hinge"/>
+        <actuator name="${lr}Motor">
+          <hardwareInterface>EffortJointInterface</hardwareInterface>
+          <mechanicalReduction>10</mechanicalReduction>
+        </actuator>
+      </transmission-->
+     </macro>
 </robot>

File: src/rosie_description/urdf/rosie.xacro (robot description, xacro)
@@ -1,6 +1,15 @@
 <?xml version='1.0'?>
 <robot name="rosie" xmlns:xacro="http://www.ros.org/wiki/xacro">
-  <xacro:property name="cameraSize" value="0.05"/>
-  <xacro:property name="cameraMass" value="0.1"/>
+  <xacro:property name="PI" value="3.1415926535897931"/>
+  <xacro:property name="chassisHeight" value="0.075"/>
+  <xacro:property name="chassisRadius" value="0.2"/>
+  <xacro:property name="chassisMass" value="4"/>
+  <xacro:property name="groundClearance" value="0.01"/>
+  <xacro:property name="casterRadius" value="0.01"/>
+  <xacro:property name="casterMass" value="0.025"/>
+  <xacro:property name="wheelRadius" value="0.032"/>
+  <xacro:property name="wheelWidth" value="0.02"/>
+  <xacro:property name="wheelBase" value="0.3"/>
+  <xacro:property name="wheelMass" value="0.05"/>
   <xacro:include filename="$(find rosie_description)/urdf/rosie.gazebo" />
   <xacro:include filename="$(find rosie_description)/urdf/materials.xacro" />
@@ -8,152 +17,47 @@
   <link name='base_link'>
     <inertial>
-      <mass value="2.0"/>
-      <!-- Assume Moment of inertia is from a solid cylinder for now -->
-	  <inertia
-          ixx="0.0209" ixy="0" ixz="0"
-          iyy="0.0209" iyz="0"
-          izz="0.04"
-      />
+      <origin xyz="0 0 0" rpy="0 0 0"/>
+      <mass value="${chassisMass}"/>
+      <cylinder_inertia m="${chassisMass}" r="${chassisRadius}" h="${chassisHeight}"/>
     </inertial>
     <collision name='collision'>
+      <origin xyz="0 0 0" rpy="0 0 0"/>
       <geometry>
-        <cylinder radius="0.2" length="0.075"/>
+        <cylinder radius="${chassisRadius}" length="${chassisHeight}"/>
       </geometry>
     </collision>
     <visual name='base_link_visual'>
+      <origin xyz="0 0 0" rpy="0 0 0"/>
       <geometry>
-        <cylinder radius="0.2" length="0.075"/>
+        <cylinder radius="${chassisRadius}" length="${chassisHeight}"/>
       </geometry>
     </visual>
   </link>
-  <link name='caster'>
-    <inertial>
-      <mass value="0.010"/>
-	  <inertia
-          ixx="0.0" ixy="0" ixz="0"
-          iyy="0.0" iyz="0"
-          izz="0.0"
-      />
-    </inertial>
-    <visual name='caster_visual'>
+  <link name="caster_wheel">
+    <collision>
+      <origin xyz="${2*casterRadius-chassisRadius} 0 ${casterRadius-(chassisHeight/2+groundClearance)}" rpy="0 0 0"/>
       <geometry>
-        <sphere radius="0.01"/>
-      </geometry>
-    </visual>
-    <collision name='collision'>
-      <geometry>
-        <sphere radius="0.01"/>
-      </geometry>
-      <!--surface>
-        <friction>
-          <ode>
-            <mu>0</mu>
-            <mu2>0</mu2>
-            <slip1>1.0</slip1>
-            <slip2>1.0</slip2>
-          </ode>
-        </friction>
-      </surface-->
-    </collision>
-  </link>
-  <joint type="fixed" name="caster_joint">
-    <origin xyz="-0.15 0 -0.0375" rpy="0 0 0"/>
-    <child link="caster"/>
-    <parent link="base_link"/>
-  </joint>
-  <link name="left_wheel">
-    <collision name="collision">
-      <origin xyz="0 0 0" rpy="0 1.5707 1.5707"/>
-      <geometry>
-        <cylinder radius="0.032" length="0.02"/>
+        <sphere radius="${casterRadius}"/>
       </geometry>
     </collision>
-    <visual name="left_wheel_visual">
-      <origin xyz="0 0 0" rpy="0 1.5707 1.5707"/>
+    <visual>
+      <origin xyz="${2*casterRadius-chassisRadius} 0 ${casterRadius-(chassisHeight/2+groundClearance)}" rpy="0 0 0"/>
       <geometry>
-        <cylinder radius="0.032" length="0.02"/>
+        <sphere radius="${casterRadius}"/>
       </geometry>
     </visual>
     <inertial>
-      <origin xyz="0 0 0" rpy="0 1.5707 1.5707"/>
-      <mass value="5"/>
-      <inertia
-        ixx=".01167" ixy="0.0" ixz="0.0"
-        iyy=".01167" iyz="0.0"
-        izz=".01885"/>
+      <origin xyz="${2*casterRadius-chassisRadius} 0 ${casterRadius-(chassisHeight/2+groundClearance)}" rpy="0 0 0"/>
+        <mass value="${casterMass}"/>
+      <sphere_inertia m="${casterMass}" r="${casterRadius}"/>
     </inertial>
   </link>
-  <joint type="continuous" name="left_wheel_hinge">
-    <origin xyz="0.05 0.15 -0.0145" rpy="0 0 0"/>
-    <child link="left_wheel"/>
+  <joint type="fixed" name="caster_wheel_joint">
+    <child link="caster_wheel"/>
     <parent link="base_link"/>
-    <axis xyz="0 1 0" rpy="0 0 0"/>
-    <limit effort="10000" velocity="1000"/>
-    <joint_properties damping="1.0" friction="1.0"/>
   </joint>
-  <link name="right_wheel">
-    <collision name="collision">
-      <origin xyz="0 0 0" rpy="0 1.5707 1.5707"/>
-      <geometry>
-        <cylinder radius="0.032" length="0.02"/>
-      </geometry>
-    </collision>
-    <visual name="right_wheel_visual">
-      <origin xyz="0 0 0" rpy="0 1.5707 1.5707"/>
-      <geometry>
-        <cylinder radius="0.032" length="0.02"/>
-      </geometry>
-    </visual>
-    <inertial>
-      <origin xyz="0 0 0" rpy="0 1.5707 1.5707"/>
-      <mass value="5"/>
-      <inertia
-        ixx=".01167" ixy="0.0" ixz="0.0"
-        iyy=".01167" iyz="0.0"
-        izz=".01885"/>
-    </inertial>
-  </link>
-  <joint type="continuous" name="right_wheel_hinge">
-    <origin xyz="0.05 -0.15 -0.0145" rpy="0 0 0"/>
-    <child link="right_wheel"/>
-    <parent link="base_link"/>
-    <axis xyz="0 1 0" rpy="0 0 0"/>
-    <limit effort="10000" velocity="1000"/>
-    <joint_properties damping="1.0" friction="1.0"/>
-  </joint>
-  <!--link name="camera">
-    <collision>
-      <origin xyz="0 0 0" rpy="0 0 0"/>
-      <geometry>
-        <box size="${cameraSize} ${cameraSize} ${cameraSize}"/>
-      </geometry>
-    </collision>
-    <visual>
-      <origin xyz="0 0 0" rpy="0 0 0"/>
-      <geometry>
-        <box size="${cameraSize} ${cameraSize} ${cameraSize}"/>
-      </geometry>
-      <material name="green"/>
-    </visual>
-    <inertial>
-      <mass value="${cameraMass}" />
-      <origin xyz="0 0 0" rpy="0 0 0"/>
-      <box_inertia m="${cameraMass}" x="${cameraSize}" y="${cameraSize}" z="${cameraSize}" />
-      <inertia ixx="1e-6" ixy="0" ixz="0" iyy="1e-6" iyz="0" izz="1e-6" />
-    </inertial>
-  </link>
-  <joint name="camera_joint" type="fixed">
-    <axis xyz="0 1 0" />
-    <origin xyz=".2 0 0" rpy="0 0 0"/>
-    <parent link="base_link"/>
-    <child link="camera"/>
-  </joint-->
-  <joint name="hokuyo_joint" type="fixed">
-    <axis xyz="0 1 0" />
-    <origin xyz="0 0 .075" rpy="0 0 0"/>
-    <parent link="base_link"/>
-    <child link="hokuyo"/>
-  </joint>
-  <!-- Hokuyo Laser -->
+  <wheel lr="left" tY="1"/>
+  <wheel lr="right" tY="-1"/>
+<!-- Hokuyo Laser -->
   <link name="hokuyo">
     <collision>
@@ -175,3 +79,34 @@
     </inertial>
   </link>
+  <joint name="hokuyo_joint" type="fixed">
+    <axis xyz="0 1 0" />
+    <origin xyz="-.05 0 .075" rpy="0 0 0"/>
+    <parent link="base_link"/>
+    <child link="hokuyo"/>
+  </joint>
+<!-- IMU -->
+  <link name="imu_link">
+    <collision>
+      <origin xyz="0 0 0" rpy="0 0 0"/>
+      <geometry>
+    <box size="0.1 0.1 0.1"/>
+      </geometry>
+    </collision>
+    <visual>
+      <origin xyz="0 0 0" rpy="0 0 0"/>
+      <geometry>
+        <box size=".025 .025 .025" />
+      </geometry>
+    </visual>
+    <inertial>
+      <mass value="1e-5" />
+      <origin xyz="0 0 0" rpy="0 0 0"/>
+      <inertia ixx="1e-6" ixy="0" ixz="0" iyy="1e-6" iyz="0" izz="1e-6" />
+    </inertial>
+  </link>
+  <joint name="imu_joint" type="fixed">
+    <origin xyz=".05 0 .0325" rpy="0 0 0"/>
+    <parent link="base_link"/>
+    <child link="imu_link"/>
+  </joint>
 </robot>
