Commit message: changed to smaller square chassis

File: src/rosie_description/urdf/macros.xacro (robot description, xacro)
@@ -48,5 +48,5 @@
           <parent link="base_link"/>
           <child link="${lr}_wheel"/>
-          <origin xyz="${+wheelBase/2-chassisRadius/2} ${tY*wheelBase/2} ${wheelRadius-(chassisHeight/2+groundClearance)}" rpy="0 0 0" />
+          <origin xyz="${-2*wheelRadius+chassisLength/2} ${tY*wheelBase/2} ${wheelRadius-(chassisHeight/2+groundClearance)}" rpy="0 0 0" />
           <axis xyz="0 1 0" rpy="0 0 0" />
           <limit effort="100" velocity="100"/>

File: src/rosie_description/urdf/rosie.xacro (robot description, xacro)
@@ -3,5 +3,6 @@
   <xacro:property name="PI" value="3.1415926535897931"/>
   <xacro:property name="chassisHeight" value="0.075"/>
-  <xacro:property name="chassisRadius" value="0.2"/>
+  <xacro:property name="chassisWidth" value="0.25"/>
+  <xacro:property name="chassisLength" value="0.3"/>
   <xacro:property name="chassisMass" value="4"/>
   <xacro:property name="groundClearance" value="0.01"/>
@@ -10,5 +11,5 @@
   <xacro:property name="wheelRadius" value="0.032"/>
   <xacro:property name="wheelWidth" value="0.02"/>
-  <xacro:property name="wheelBase" value="0.3"/>
+  <xacro:property name="wheelBase" value="0.2"/>
   <xacro:property name="wheelMass" value="0.05"/>
   <xacro:include filename="$(find rosie_description)/urdf/rosie.gazebo" />
@@ -19,10 +20,10 @@
       <origin xyz="0 0 0" rpy="0 0 0"/>
       <mass value="${chassisMass}"/>
-      <cylinder_inertia m="${chassisMass}" r="${chassisRadius}" h="${chassisHeight}"/>
+      <box_inertia m="${chassisMass}" x="${chassisLength}" y="${chassisWidth}" z="${chassisHeight}"/>
     </inertial>
     <collision name='collision'>
       <origin xyz="0 0 0" rpy="0 0 0"/>
       <geometry>
-        <cylinder radius="${chassisRadius}" length="${chassisHeight}"/>
+        <box size="${chassisLength} ${chassisWidth} ${chassisHeight}"/>
       </geometry>
     </collision>
@@ -30,5 +31,5 @@
       <origin xyz="0 0 0" rpy="0 0 0"/>
       <geometry>
-        <cylinder radius="${chassisRadius}" length="${chassisHeight}"/>
+        <box size="${chassisLength} ${chassisWidth} ${chassisHeight}"/>
       </geometry>
     </visual>
@@ -36,5 +37,5 @@
   <link name="caster_wheel">
     <collision>
-      <origin xyz="${2*casterRadius-chassisRadius} 0 ${casterRadius-(chassisHeight/2+groundClearance)}" rpy="0 0 0"/>
+      <origin xyz="${2*casterRadius-chassisLength/2} 0 ${casterRadius-(chassisHeight/2+groundClearance)}" rpy="0 0 0"/>
       <geometry>
         <sphere radius="${casterRadius}"/>
@@ -42,5 +43,5 @@
     </collision>
     <visual>
-      <origin xyz="${2*casterRadius-chassisRadius} 0 ${casterRadius-(chassisHeight/2+groundClearance)}" rpy="0 0 0"/>
+      <origin xyz="${2*casterRadius-chassisLength/2} 0 ${casterRadius-(chassisHeight/2+groundClearance)}" rpy="0 0 0"/>
       <geometry>
         <sphere radius="${casterRadius}"/>
@@ -48,5 +49,5 @@
     </visual>
     <inertial>
-      <origin xyz="${2*casterRadius-chassisRadius} 0 ${casterRadius-(chassisHeight/2+groundClearance)}" rpy="0 0 0"/>
+      <origin xyz="${2*casterRadius-chassisLength/2} 0 ${casterRadius-(chassisHeight/2+groundClearance)}" rpy="0 0 0"/>
         <mass value="${casterMass}"/>
       <sphere_inertia m="${casterMass}" r="${casterRadius}"/>
@@ -81,5 +82,5 @@
   <joint name="hokuyo_joint" type="fixed">
     <axis xyz="0 1 0" />
-    <origin xyz="-.05 0 .075" rpy="0 0 0"/>
+    <origin xyz="-.05 0 .05" rpy="0 0 0"/>
     <parent link="base_link"/>
     <child link="hokuyo"/>

Commit message: updated to reflect CAD values

File: src/rosie_description/urdf/macros.xacro (robot description, xacro)
@@ -48,5 +48,5 @@
           <parent link="base_link"/>
           <child link="${lr}_wheel"/>
-          <origin xyz="${-2*wheelRadius+chassisLength/2} ${tY*wheelBase/2} ${wheelRadius-(chassisHeight/2+groundClearance)}" rpy="0 0 0" />
+          <origin xyz=".05 ${tY*wheelBase/2} ${wheelRadius-(chassisHeight/2+groundClearance)}" rpy="0 0 0" />
           <axis xyz="0 1 0" rpy="0 0 0" />
           <limit effort="100" velocity="100"/>

File: src/rosie_description/urdf/rosie.xacro (robot description, xacro)
@@ -2,14 +2,14 @@
 <robot name="rosie" xmlns:xacro="http://www.ros.org/wiki/xacro">
   <xacro:property name="PI" value="3.1415926535897931"/>
-  <xacro:property name="chassisHeight" value="0.075"/>
-  <xacro:property name="chassisWidth" value="0.25"/>
+  <xacro:property name="chassisHeight" value="0.060"/>
+  <xacro:property name="chassisWidth" value="0.240"/>
   <xacro:property name="chassisLength" value="0.3"/>
   <xacro:property name="chassisMass" value="4"/>
   <xacro:property name="groundClearance" value="0.01"/>
-  <xacro:property name="casterRadius" value="0.01"/>
+  <xacro:property name="casterRadius" value="0.02"/>
   <xacro:property name="casterMass" value="0.025"/>
-  <xacro:property name="wheelRadius" value="0.032"/>
-  <xacro:property name="wheelWidth" value="0.02"/>
-  <xacro:property name="wheelBase" value="0.2"/>
+  <xacro:property name="wheelRadius" value="0.030"/>
+  <xacro:property name="wheelWidth" value="0.025"/>
+  <xacro:property name="wheelBase" value="0.185"/>
   <xacro:property name="wheelMass" value="0.05"/>
   <xacro:include filename="$(find rosie_description)/urdf/rosie.gazebo" />
@@ -37,5 +37,5 @@
   <link name="caster_wheel">
     <collision>
-      <origin xyz="${2*casterRadius-chassisLength/2} 0 ${casterRadius-(chassisHeight/2+groundClearance)}" rpy="0 0 0"/>
+      <origin xyz="-0.125 0 ${casterRadius-(chassisHeight/2+groundClearance)}" rpy="0 0 0"/>
       <geometry>
         <sphere radius="${casterRadius}"/>
@@ -43,5 +43,5 @@
     </collision>
     <visual>
-      <origin xyz="${2*casterRadius-chassisLength/2} 0 ${casterRadius-(chassisHeight/2+groundClearance)}" rpy="0 0 0"/>
+      <origin xyz="-0.125 0 ${casterRadius-(chassisHeight/2+groundClearance)}" rpy="0 0 0"/>
       <geometry>
         <sphere radius="${casterRadius}"/>
@@ -49,5 +49,5 @@
     </visual>
     <inertial>
-      <origin xyz="${2*casterRadius-chassisLength/2} 0 ${casterRadius-(chassisHeight/2+groundClearance)}" rpy="0 0 0"/>
+      <origin xyz="-0.125 0 ${casterRadius-(chassisHeight/2+groundClearance)}" rpy="0 0 0"/>
         <mass value="${casterMass}"/>
       <sphere_inertia m="${casterMass}" r="${casterRadius}"/>
@@ -82,5 +82,5 @@
   <joint name="hokuyo_joint" type="fixed">
     <axis xyz="0 1 0" />
-    <origin xyz="-.05 0 .05" rpy="0 0 0"/>
+    <origin xyz=".07 0 .06" rpy="0 0 0"/>
     <parent link="base_link"/>
     <child link="hokuyo"/>
@@ -91,5 +91,5 @@
       <origin xyz="0 0 0" rpy="0 0 0"/>
       <geometry>
-    <box size="0.1 0.1 0.1"/>
+    <box size="0.01 0.01 0.01"/>
       </geometry>
     </collision>
@@ -97,5 +97,5 @@
       <origin xyz="0 0 0" rpy="0 0 0"/>
       <geometry>
-        <box size=".025 .025 .025" />
+        <box size="0.01 0.01 0.01" />
       </geometry>
     </visual>
@@ -107,5 +107,5 @@
   </link>
   <joint name="imu_joint" type="fixed">
-    <origin xyz=".05 0 .0325" rpy="0 0 0"/>
+    <origin xyz="0.08 0.050 -0.01" rpy="0 0 0"/>
     <parent link="base_link"/>
     <child link="imu_link"/>
