Commit message: amcl and move_base demo working

File: src/rosie_description/urdf/rosie.xacro (robot description, xacro)
@@ -1,4 +1,6 @@
 <?xml version='1.0'?>
-<robot name="rosie" xmlns:xacro="http://www.ros.org/wiki/xacro">
+<robot name="myrobot" xmlns:xacro="http://www.ros.org/wiki/xacro">
+  <xacro:property name="cameraSize" value="0.05"/>
+  <xacro:property name="cameraMass" value="0.1"/>
   <xacro:include filename="$(find rosie_description)/urdf/rosie.gazebo" />
   <xacro:include filename="$(find rosie_description)/urdf/materials.xacro" />
@@ -7,9 +9,9 @@
     <pose>0 0 0.1 0 0 0</pose>
     <inertial>
-      <mass value="10.0"/>
+      <mass value="15.0"/>
       <origin xyz="0.0 0 0.1" rpy=" 0 0 0"/>
       <inertia
-          ixx="0.5" ixy="0" ixz="0"
-          iyy="1.0" iyz="0"
+          ixx="0.1" ixy="0" ixz="0"
+          iyy="0.1" iyz="0"
           izz="0.1"
       />
@@ -17,5 +19,5 @@
     <collision name='collision'>
       <geometry>
-        <box size=".19 .19 .05"/>
+        <box size=".4 .2 .1"/>
       </geometry>
     </collision>
@@ -23,11 +25,11 @@
       <origin xyz="0 0 0" rpy=" 0 0 0"/>
       <geometry>
-        <box size=".19 .19 .05"/>
+        <box size=".4 .2 .1"/>
       </geometry>
     </visual>
     <collision name='caster_collision'>
-      <origin xyz="0.11 0 -0.025" rpy=" 0 0 0"/>
+      <origin xyz="-0.15 0 -0.05" rpy=" 0 0 0"/>
       <geometry>
-        <sphere radius="0.01"/>
+        <sphere radius="0.05"/>
       </geometry>
       <surface>
@@ -43,7 +45,29 @@
     </collision>
     <visual name='caster_visual'>
-      <origin xyz="0.11 0 -0.025" rpy=" 0 0 0"/>
+      <origin xyz="-0.15 0 -0.05" rpy=" 0 0 0"/>
       <geometry>
-        <sphere radius="0.01"/>
+        <sphere radius="0.05"/>
+      </geometry>
+    </visual>
+    <collision name='caster_front_collision'>
+      <origin xyz="0.15 0 -0.05" rpy=" 0 0 0"/>
+      <geometry>
+        <sphere radius="0.05"/>
+      </geometry>
+      <surface>
+        <friction>
+          <ode>
+            <mu>0</mu>
+            <mu2>0</mu2>
+            <slip1>1.0</slip1>
+            <slip2>1.0</slip2>
+          </ode>
+        </friction>
+      </surface>
+    </collision>
+    <visual name='caster_front_visual'>
+      <origin xyz="0.15 0 -0.05" rpy=" 0 0 0"/>
+      <geometry>
+        <sphere radius="0.05"/>
       </geometry>
     </visual>
@@ -54,5 +78,5 @@
       <origin xyz="0 0 0" rpy="0 1.5707 1.5707"/>
       <geometry>
-        <cylinder radius="0.04" length="0.01"/>
+        <cylinder radius="0.1" length="0.05"/>
       </geometry>
     </collision>
@@ -60,5 +84,5 @@
       <origin xyz="0 0 0" rpy="0 1.5707 1.5707"/>
       <geometry>
-        <cylinder radius="0.04" length="0.01"/>
+        <cylinder radius="0.1" length="0.05"/>
       </geometry>
     </visual>
@@ -66,9 +90,8 @@
       <origin xyz="0 0 0" rpy="0 1.5707 1.5707"/>
       <mass value="5"/>
-      <cylinder_inertia m="5" r="0.04" h="0.01"/>
       <inertia
-        ixx="1.0" ixy="0.0" ixz="0.0"
-        iyy="1.0" iyz="0.0"
-        izz="1.0"/>
+        ixx=".1" ixy="0.0" ixz="0.0"
+        iyy=".1" iyz="0.0"
+        izz=".1"/>
     </inertial>
   </link>
@@ -78,5 +101,5 @@
       <origin xyz="0 0 0" rpy="0 1.5707 1.5707"/>
       <geometry>
-        <cylinder radius="0.04" length="0.01"/>
+        <cylinder radius="0.1" length="0.05"/>
       </geometry>
     </collision>
@@ -84,5 +107,5 @@
       <origin xyz="0 0 0" rpy="0 1.5707 1.5707"/>
       <geometry>
-        <cylinder radius="0.04" length="0.01"/>
+        <cylinder radius="0.1" length="0.05"/>
       </geometry>
     </visual>
@@ -90,26 +113,80 @@
       <origin xyz="0 0 0" rpy="0 1.5707 1.5707"/>
       <mass value="5"/>
-      <cylinder_inertia m="5" r="0.04" h="0.01"/>
       <inertia
-        ixx="1.0" ixy="0.0" ixz="0.0"
-        iyy="1.0" iyz="0.0"
-        izz="1.0"/>
+        ixx=".1" ixy="0.0" ixz="0.0"
+        iyy=".1" iyz="0.0"
+        izz=".1"/>
     </inertial>
   </link>
   <joint type="continuous" name="left_wheel_hinge">
-    <origin xyz="-0.045 0.09 0" rpy="0 0 0"/>
+    <origin xyz="0 0.15 0" rpy="0 0 0"/>
+    <!--origin xyz="0.1 0.13 0" rpy="0 1.5707 1.5707"/-->
     <child link="left_wheel"/>
     <parent link="chassis"/>
     <axis xyz="0 1 0" rpy="0 0 0"/>
-    <limit effort="100" velocity="100"/>
-    <joint_properties damping="0.0" friction="0.0"/>
+    <limit effort="10000" velocity="1000"/>
+    <joint_properties damping="1.0" friction="1.0"/>
   </joint>
   <joint type="continuous" name="right_wheel_hinge">
-    <origin xyz="-0.045 -0.09 0" rpy="0 0 0"/>
+    <origin xyz="0 -0.15 0" rpy="0 0 0"/>
+    <!--origin xyz="0.1 -0.13 0" rpy="0 1.5707 1.5707"/-->
     <child link="right_wheel"/>
     <parent link="chassis"/>
     <axis xyz="0 1 0" rpy="0 0 0"/>
-    <limit effort="100" velocity="100"/>
-    <joint_properties damping="0.0" friction="0.0"/>
+    <limit effort="10000" velocity="1000"/>
+    <joint_properties damping="1.0" friction="1.0"/>
   </joint>
+  <link name="camera">
+    <collision>
+      <origin xyz="0 0 0" rpy="0 0 0"/>
+      <geometry>
+        <box size="${cameraSize} ${cameraSize} ${cameraSize}"/>
+      </geometry>
+    </collision>
+    <visual>
+      <origin xyz="0 0 0" rpy="0 0 0"/>
+      <geometry>
+        <box size="${cameraSize} ${cameraSize} ${cameraSize}"/>
+      </geometry>
+      <material name="green"/>
+    </visual>
+    <inertial>
+      <mass value="${cameraMass}" />
+      <origin xyz="0 0 0" rpy="0 0 0"/>
+      <box_inertia m="${cameraMass}" x="${cameraSize}" y="${cameraSize}" z="${cameraSize}" />
+      <inertia ixx="1e-6" ixy="0" ixz="0" iyy="1e-6" iyz="0" izz="1e-6" />
+    </inertial>
+  </link>
+  <joint name="camera_joint" type="fixed">
+    <axis xyz="0 1 0" />
+    <origin xyz=".2 0 0" rpy="0 0 0"/>
+    <parent link="chassis"/>
+    <child link="camera"/>
+  </joint>
+  <joint name="hokuyo_joint" type="fixed">
+    <axis xyz="0 1 0" />
+    <origin xyz=".15 0 .1" rpy="0 0 0"/>
+    <parent link="chassis"/>
+    <child link="hokuyo"/>
+  </joint>
+  <!-- Hokuyo Laser -->
+  <link name="hokuyo">
+    <collision>
+      <origin xyz="0 0 0" rpy="0 0 0"/>
+      <geometry>
+    <box size="0.1 0.1 0.1"/>
+      </geometry>
+    </collision>
+    <visual>
+      <origin xyz="0 0 0" rpy="0 0 0"/>
+      <geometry>
+        <mesh filename="package://rosie_description/meshes/hokuyo.dae"/>
+      </geometry>
+    </visual>
+    <inertial>
+      <mass value="1e-5" />
+      <origin xyz="0 0 0" rpy="0 0 0"/>
+      <inertia ixx="1e-6" ixy="0" ixz="0" iyy="1e-6" iyz="0" izz="1e-6" />
+    </inertial>
+  </link>
 </robot>

Commit message: rotated scanner frame

File: src/rosie_description/urdf/rosie.xacro (robot description, xacro)
@@ -82,5 +82,5 @@
   <joint name="hokuyo_joint" type="fixed">
     <axis xyz="0 1 0" />
-    <origin xyz=".07 0 .06" rpy="0 0 0"/>
+    <origin xyz=".07 0 .06" rpy="0 0 3.14159"/>
     <parent link="base_link"/>
     <child link="hokuyo"/>

Commit message: adjusted resolution

File: src/rosie_description/urdf/rosie.xacro (robot description, xacro)
@@ -81,5 +81,5 @@
   </link>
   <joint name="hokuyo_joint" type="fixed">
-    <axis xyz="0 1 0" />
+    <!--axis xyz="0 1 0" />-->
     <origin xyz=".07 0 .06" rpy="0 0 3.14159"/>
     <parent link="base_link"/>

Commit message: set hokuyo rotation to 0

File: src/rosie_description/urdf/rosie.xacro (robot description, xacro)
@@ -82,5 +82,5 @@
   <joint name="hokuyo_joint" type="fixed">
     <!--axis xyz="0 1 0" />-->
-    <origin xyz=".07 0 .06" rpy="0 0 3.14159"/>
+    <origin xyz=".07 0 .06" rpy="0 0 0"/>
     <parent link="base_link"/>
     <child link="hokuyo"/>

Commit message: set hokuyo rotation to 0.6981

File: src/rosie_description/urdf/rosie.xacro (robot description, xacro)
@@ -82,5 +82,5 @@
   <joint name="hokuyo_joint" type="fixed">
     <!--axis xyz="0 1 0" />-->
-    <origin xyz=".07 0 .06" rpy="0 0 0"/>
+    <origin xyz=".07 0 .06" rpy="0 0 0.698132"/>
     <parent link="base_link"/>
     <child link="hokuyo"/>

Commit message: changed reconstructed laser message frame to hokuyo

File: src/rosie_description/urdf/rosie.xacro (robot description, xacro)
@@ -82,5 +82,5 @@
   <joint name="hokuyo_joint" type="fixed">
     <!--axis xyz="0 1 0" />-->
-    <origin xyz=".07 0 .06" rpy="0 0 0.698132"/>
+    <origin xyz=".07 0 .06" rpy="0 0 -0.698132"/>
     <parent link="base_link"/>
     <child link="hokuyo"/>

Commit message: changed nav params

File: src/rosie_description/urdf/rosie.xacro (robot description, xacro)
@@ -82,5 +82,5 @@
   <joint name="hokuyo_joint" type="fixed">
     <!--axis xyz="0 1 0" />-->
-    <origin xyz=".07 0 .06" rpy="0 0 -0.698132"/>
+    <origin xyz=".07 0 .06" rpy="0 0 0"/>
     <parent link="base_link"/>
     <child link="hokuyo"/>

Commit message: changed nav params

File: src/rosie_description/urdf/rosie.xacro (robot description, xacro)
@@ -107,5 +107,5 @@
   </link>
   <joint name="imu_joint" type="fixed">
-    <origin xyz="0.08 0.050 -0.01" rpy="0 0 0"/>
+    <origin xyz="0.045 -0.070 -0.01" rpy="0 0 0"/>
     <parent link="base_link"/>
     <child link="imu_link"/>

Commit message: null

File: src/rosie_description/urdf/rosie.xacro (robot description, xacro)
@@ -107,5 +107,5 @@
   </link>
   <joint name="imu_joint" type="fixed">
-    <origin xyz="0.045 -0.070 -0.01" rpy="0 0 0"/>
+    <origin xyz="-0.070 -0.045 -0.01" rpy="0 0 0"/>
     <parent link="base_link"/>
     <child link="imu_link"/>

Commit message: increased laser max range and fixed URDF to match robot

File: src/rosie_description/urdf/rosie.xacro (robot description, xacro)
@@ -2,14 +2,14 @@
 <robot name="rosie" xmlns:xacro="http://www.ros.org/wiki/xacro">
   <xacro:property name="PI" value="3.1415926535897931"/>
-  <xacro:property name="chassisHeight" value="0.060"/>
-  <xacro:property name="chassisWidth" value="0.240"/>
-  <xacro:property name="chassisLength" value="0.3"/>
+  <xacro:property name="chassisHeight" value="0.095"/>
+  <xacro:property name="chassisWidth" value="0.250"/>
+  <xacro:property name="chassisLength" value="0.250"/>
   <xacro:property name="chassisMass" value="4"/>
   <xacro:property name="groundClearance" value="0.01"/>
-  <xacro:property name="casterRadius" value="0.02"/>
+  <xacro:property name="casterRadius" value="0.025"/>
   <xacro:property name="casterMass" value="0.025"/>
-  <xacro:property name="wheelRadius" value="0.030"/>
-  <xacro:property name="wheelWidth" value="0.025"/>
-  <xacro:property name="wheelBase" value="0.185"/>
+  <xacro:property name="wheelRadius" value="0.040"/>
+  <xacro:property name="wheelWidth" value="0.020"/>
+  <xacro:property name="wheelBase" value="0.200"/>
   <xacro:property name="wheelMass" value="0.05"/>
   <xacro:include filename="$(find rosie_description)/urdf/rosie.gazebo" />
@@ -37,5 +37,5 @@
   <link name="caster_wheel">
     <collision>
-      <origin xyz="-0.125 0 ${casterRadius-(chassisHeight/2+groundClearance)}" rpy="0 0 0"/>
+      <origin xyz="-0.145 0 ${casterRadius-(chassisHeight/2+groundClearance)}" rpy="0 0 0"/>
       <geometry>
         <sphere radius="${casterRadius}"/>
@@ -82,5 +82,5 @@
   <joint name="hokuyo_joint" type="fixed">
     <!--axis xyz="0 1 0" />-->
-    <origin xyz=".07 0 .06" rpy="0 0 0"/>
+    <origin xyz=".05 0 .12" rpy="0 0 0"/>
     <parent link="base_link"/>
     <child link="hokuyo"/>
@@ -107,5 +107,5 @@
   </link>
   <joint name="imu_joint" type="fixed">
-    <origin xyz="-0.070 -0.045 -0.01" rpy="0 0 0"/>
+    <origin xyz="-0.040 -0.085 -0.03" rpy="0 0 0"/>
     <parent link="base_link"/>
     <child link="imu_link"/>
